File: Hardware/Asgard/kicad/PCB/PCB.sch (KiCad schematic (older format))
At the start: 0 parts

Commit message: Updated Template Kicad
Parts:
- added U1: Teensy3.6, symbol Teensy3.6
Changed lines of the file:
@@
 LIBS:contrib
 LIBS:valves
-LIBS:teensy_3.1
+LIBS:teensy
+LIBS:PCB-cache
 EELAYER 25 0
 EELAYER END
@@
 EndData
 $EndBitmap
+$Comp
+L Teensy3.6 U1
+U 1 1 58D92D6F
+P 4000 3500
+F 0 "U1" H 4000 5800 60  0000 C CNN
+F 1 "Teensy3.6" H 4000 1200 60  0000 C CNN
+F 2 "" H 4000 3500 60  0000 C CNN
+F 3 "" H 4000 3500 60  0000 C CNN
+	1    4000 3500
+	1    0    0    -1
+$EndComp
 $EndSCHEMATC
