File: Hardware/Asgard/kicad/Asgard/Asgard.sch (KiCad schematic (older format))
At the start: 1 part, among them U1 Teensy3.6

Commit message: template
Parts:
- removed U1: Teensy3.6, symbol Teensy3.6
- added U?: Teensy3.6, symbol Teensy3.6
Changed lines of the file:
@@
 LIBS:valves
 LIBS:teensy
-LIBS:PCB-cache
+LIBS:Asgard-cache
 EELAYER 25 0
 EELAYER END
@@
 $EndBitmap
 $Comp
-L Teensy3.6 U1
-U 1 1 58D92D6F
-P 4000 3500
-F 0 "U1" H 4000 5800 60  0000 C CNN
-F 1 "Teensy3.6" H 4000 1200 60  0000 C CNN
-F 2 "" H 4000 3500 60  0000 C CNN
-F 3 "" H 4000 3500 60  0000 C CNN
-	1    4000 3500
+L Teensy3.6 U?
+U 1 1 58D930E1
+P 2650 3550
+F 0 "U?" H 2650 5850 60  0000 C CNN
+F 1 "Teensy3.6" H 2650 1250 60  0000 C CNN
+F 2 "" H 2650 3550 60  0000 C CNN
+F 3 "" H 2650 3550 60  0000 C CNN
+	1    2650 3550
 	1    0    0    -1
 $EndComp

Commit message: gg
Parts:
- added J? (x2): CONN_01X04, symbol CONN_01X04
- added J?: CONN_01X06, symbol CONN_01X06
Changed lines of the file:
@@
+	1    0    0    -1
+$EndComp
+$Comp
+L CONN_01X04 J?
+U 1 1 58D93201
+P 6500 1800
+F 0 "J?" H 6500 2050 50  0000 C CNN
+F 1 "CONN_01X04" V 6600 1800 50  0000 C CNN
+F 2 "" H 6500 1800 50  0001 C CNN
+F 3 "" H 6500 1800 50  0001 C CNN
+	1    6500 1800
+	1    0    0    -1
+$EndComp
+$Comp
+L CONN_01X04 J?
+U 1 1 58D93258
+P 6500 2550
+F 0 "J?" H 6500 2800 50  0000 C CNN
+F 1 "CONN_01X04" V 6600 2550 50  0000 C CNN
+F 2 "" H 6500 2550 50  0001 C CNN
+F 3 "" H 6500 2550 50  0001 C CNN
+	1    6500 2550
+	1    0    0    -1
+$EndComp
+$Comp
+L CONN_01X06 J?
+U 1 1 58D932F8
+P 6550 3450
+F 0 "J?" H 6550 3800 50  0000 C CNN
+F 1 "CONN_01X06" V 6650 3450 50  0000 C CNN
+F 2 "" H 6550 3450 50  0001 C CNN
+F 3 "" H 6550 3450 50  0001 C CNN
+	1    6550 3450
 	1    0    0    -1
 $EndComp

Commit message: Initial setup of Kicad
Libraries setup
Parts:
- removed U?: Teensy3.6, symbol Teensy3.6
- added U1: Teensy3.6fsocket, Teensy:Socket_Strip_Teensy3.6_2x24_Pitch2.54mm, symbol Teensy3.6fsocket
- J1, J2: renamed from J?; footprint (none) -> Socket_Strips:Socket_Strip_Angled_1x04_Pitch2.54mm
- J3: renamed from J?; footprint (none) -> Socket_Strips:Socket_Strip_Straight_1x06_Pitch2.54mm
Connections:
- wire segments 0 -> 3
Changed lines of the file:
@@
 $Bitmap
 Pos 7250 6800
-Scale 1.000000
+Scale 1,000000
 Data
 89 50 4E 47 0D 0A 1A 0A 00 00 00 0D 49 48 44 52 00 00 00 80 00 00 00 80 08 06 00 00 00 C3 3E 61
@@
 $EndBitmap
 $Comp
-L Teensy3.6 U?
-U 1 1 58D930E1
-P 2650 3550
-F 0 "U?" H 2650 5850 60  0000 C CNN
-F 1 "Teensy3.6" H 2650 1250 60  0000 C CNN
-F 2 "" H 2650 3550 60  0000 C CNN
-F 3 "" H 2650 3550 60  0000 C CNN
-	1    2650 3550
-	1    0    0    -1
-$EndComp
-$Comp
-L CONN_01X04 J?
+L CONN_01X04 J1
 U 1 1 58D93201
 P 6500 1800
-F 0 "J?" H 6500 2050 50  0000 C CNN
+F 0 "J1" H 6500 2050 50  0000 C CNN
 F 1 "CONN_01X04" V 6600 1800 50  0000 C CNN
-F 2 "" H 6500 1800 50  0001 C CNN
+F 2 "Socket_Strips:Socket_Strip_Angled_1x04_Pitch2.54mm" H 6500 1800 50  0001 C CNN
 F 3 "" H 6500 1800 50  0001 C CNN
 	1    6500 1800
@@
 $EndComp
 $Comp
-L CONN_01X04 J?
+L CONN_01X04 J2
 U 1 1 58D93258
 P 6500 2550
-F 0 "J?" H 6500 2800 50  0000 C CNN
+F 0 "J2" H 6500 2800 50  0000 C CNN
 F 1 "CONN_01X04" V 6600 2550 50  0000 C CNN
-F 2 "" H 6500 2550 50  0001 C CNN
+F 2 "Socket_Strips:Socket_Strip_Angled_1x04_Pitch2.54mm" H 6500 2550 50  0001 C CNN
 F 3 "" H 6500 2550 50  0001 C CNN
 	1    6500 2550
@@
 $EndComp
 $Comp
-L CONN_01X06 J?
+L CONN_01X06 J3
 U 1 1 58D932F8
 P 6550 3450
-F 0 "J?" H 6550 3800 50  0000 C CNN
+F 0 "J3" H 6550 3800 50  0000 C CNN
 F 1 "CONN_01X06" V 6650 3450 50  0000 C CNN
-F 2 "" H 6550 3450 50  0001 C CNN
+F 2 "Socket_Strips:Socket_Strip_Straight_1x06_Pitch2.54mm" H 6550 3450 50  0001 C CNN
 F 3 "" H 6550 3450 50  0001 C CNN
 	1    6550 3450
 	1    0    0    -1
 $EndComp
+$Comp
+L Teensy3.6fsocket U1
+U 1 1 58D95F25
+P 3000 3750
+F 0 "U1" H 3000 6050 60  0000 C CNN
+F 1 "Teensy3.6fsocket" H 3000 3300 60  0000 C CNN
+F 2 "Teensy:Socket_Strip_Teensy3.6_2x24_Pitch2.54mm" H 3000 3750 60  0001 C CNN
+F 3 "" H 3000 3750 60  0000 C CNN
+	1    3000 3750
+	1    0    0    -1
+$EndComp
+Wire Wire Line
+	4000 1950 6300 1950
+Wire Wire Line
+	6300 2400 4000 2400
+Wire Wire Line
+	4000 2400 4000 2450
 $EndSCHEMATC

Commit message: Proposal Asgard Schematics
Ready for routing
Parts:
- removed U1: Teensy3.6fsocket, Teensy:Socket_Strip_Teensy3.6_2x24_Pitch2.54mm, symbol Teensy3.6fsocket
- added OAT1: CONN_01X03, Pin_Headers:Pin_Header_Angled_1x03_Pitch2.54mm, symbol CONN_01X03
- added R1, R2, R3, R4: 4700, Resistors_SMD:R_1206, symbol R
- added TEENSYV3.6: Teensy3.6fsocket, Teensy:Socket_Strip_Teensy3.6_2x24_Pitch2.54mm, symbol Teensy3.6fsocket
- renumbered J2 to ABSP1, J3 to BLUESMIRF1, J1 to DELTAP1
Connections:
- wire segments 3 -> 44
Other:
- note added: "3.3V"
- note added: "ADC Asgard"
- note added: "Absolute pressure sensor\nHSCSRNN1.6BA2A3 0x28 address"
- note added: "BasicAirData"
- note added: "BlueSMiRF Bluetooth module"
- note added: "CTS"
- note added: "GND"
- note added: "Pin 1 GND, PIN 2 VS,PIN 3 SDA,PIN 4 SCL"
- note added: "RTS-0"
- note added: "RX-1"
- note added: "Realtive pressure sensor\nHSCSRRD001PD2A3"
- note added: "TX-0"
- note added: "Temperature Sensor\nTMP36GT9Z"
- note added: "VCC"
- note added: "VOUT"
- note added: "www.basicairdata.eu"
- note removed: "BasicAirData\nwww.basicairdata.eu"
- moved on the sheet: ABSP1, BLUESMIRF1, DELTAP1

Commit message: PCB Preliminary Layout
Connections:
- net labels added: +3.3V, GND
- wire segments 44 -> 46
Changed lines of the file:
@@
 	0    1    1    0
 $EndComp
-Text Notes 4300 1800 0    59   ~ 0
-3.3V
 $Comp
 L Teensy3.6fsocket TEENSYV3.6
@@
 	1    0    0    -1
 $EndComp
-Text Notes 4050 1800 0    60   ~ 0
-GND
 Wire Wire Line
 	4350 1850 4350 5750
@@
 	5000 3500 5200 3500
 Wire Wire Line
-	4150 1850 4150 5550
+	4150 1600 4150 5550
 Wire Wire Line
 	3650 2950 5150 2950
@@
 Wire Wire Line
 	3000 5550 4150 5550
+$Comp
+L GND #PWR01
+U 1 1 58DA5935
+P 3900 1650
+F 0 "#PWR01" H 3900 1400 50  0001 C CNN
+F 1 "GND" H 3900 1500 50  0000 C CNN
+F 2 "" H 3900 1650 50  0001 C CNN
+F 3 "" H 3900 1650 50  0001 C CNN
+	1    3900 1650
+	1    0    0    -1
+$EndComp
+Wire Wire Line
+	4150 1600 3900 1600
+Wire Wire Line
+	3900 1600 3900 1650
+$Comp
+L +3.3V #PWR02
+U 1 1 58DA5ABD
+P 4350 1850
+F 0 "#PWR02" H 4350 1700 50  0001 C CNN
+F 1 "+3.3V" H 4350 1990 50  0000 C CNN
+F 2 "" H 4350 1850 50  0001 C CNN
+F 3 "" H 4350 1850 50  0001 C CNN
+	1    4350 1850
+	1    0    0    -1
+$EndComp
 $EndSCHEMATC
