File: Hardware/Asgard/kicad/Asgard/Asgard.sch (KiCad schematic (older format))
At the start: 10 parts

Commit message: PCB Candidate 2
Connections:
- net at TEENSYV3.6.29 (A8): now also GPIO1.1 (P1)
- net at TEENSYV3.6.30 (A7): now also GPIO1.2 (P2)
- net at TEENSYV3.6.47 (A15): no longer GPIO1.1 (P1)
- net at TEENSYV3.6.48 (A14): no longer GPIO1.2 (P2)
Changed lines of the file:
@@
 $Bitmap
 Pos 7250 6800
-Scale 1.000000
+Scale 1,000000
 Data
 89 50 4E 47 0D 0A 1A 0A 00 00 00 0D 49 48 44 52 00 00 00 80 00 00 00 80 08 06 00 00 00 C3 3E 61
@@
 $Bitmap
 Pos 7050 5000
-Scale 1.000000
+Scale 1,000000
 Data
 89 50 4E 47 0D 0A 1A 0A 00 00 00 0D 49 48 44 52 00 00 02 58 00 00 02 58 08 02 00 00 00 31 04 0F
@@
 $Bitmap
 Pos 6800 3400
-Scale 1.000000
+Scale 1,000000
 Data
 89 50 4E 47 0D 0A 1A 0A 00 00 00 0D 49 48 44 52 00 00 02 23 00 00 01 87 08 02 00 00 00 ED 2D C5
@@
 $Bitmap
 Pos 6800 2000
-Scale 1.000000
+Scale 1,000000
 Data
 89 50 4E 47 0D 0A 1A 0A 00 00 00 0D 49 48 44 52 00 00 02 33 00 00 01 A2 08 02 00 00 00 9D E2 D0
@@
 $Bitmap
 Pos 4300 6300
-Scale 1.000000
+Scale 1,000000
 Data
 89 50 4E 47 0D 0A 1A 0A 00 00 00 0D 49 48 44 52 00 00 02 34 00 00 01 2F 08 02 00 00 00 DD 10 CC
@@
 $Bitmap
 Pos 9550 5400
-Scale 1.000000
+Scale 1,000000
 Data
 89 50 4E 47 0D 0A 1A 0A 00 00 00 0D 49 48 44 52 00 00 02 EE 00 00 02 32 08 02 00 00 00 1B 83 D8
@@
 	2400 6150 2400 5350
 Wire Wire Line
-	2400 5350 3900 5350
+	3900 5350 2400 5350
 Wire Wire Line
-	3800 5200 3800 4450
+	3900 2550 3900 5350
 Wire Wire Line
-	3800 4450 3650 4450
+	3800 5200 3800 2650
 Wire Wire Line
-	3650 4350 3900 4350
+	3800 2650 3650 2650
 Wire Wire Line
-	3900 4350 3900 5350
+	3900 2550 3650 2550
 $EndSCHEMATC

Commit message: PCB candidate 4
Connections:
- net GND: no longer GPIO1.3 (P3)
- net at TEENSYV3.6.28 (A9): now also GPIO1.1 (P1)
- net at TEENSYV3.6.29 (A8): now also GPIO1.2 (P2); no longer GPIO1.1 (P1)
- net at TEENSYV3.6.30 (A7): now also GPIO1.3 (P3); no longer GPIO1.2 (P2)
Changed lines of the file:
@@
 	4000 3350 3650 3350
 Wire Wire Line
-	3000 6150 3000 5550
-Wire Wire Line
-	3000 5550 4150 5550
+	4150 5550 3000 5550
 Wire Wire Line
 	4150 1600 3900 1600
@@
 $EndComp
 Wire Wire Line
-	2200 6150 2200 6000
-Wire Wire Line
-	2200 6000 3000 6000
-Wire Wire Line
-	3000 6000 3000 5950
-Connection ~ 3000 5950
+	2200 5150 2200 6150
 Wire Wire Line
 	3800 5200 2300 5200
@@
 	2400 6150 2400 5350
 Wire Wire Line
-	3900 5350 2400 5350
+	2400 5350 3900 5350
 Wire Wire Line
-	3900 2550 3900 5350
+	3900 5350 3900 2450
 Wire Wire Line
-	3800 5200 3800 2650
+	3800 2550 3800 5200
 Wire Wire Line
-	3800 2650 3650 2650
+	3900 2450 3650 2450
 Wire Wire Line
-	3900 2550 3650 2550
+	3800 2550 3650 2550
+Wire Wire Line
+	3000 5550 3000 6150
+Wire Wire Line
+	2200 5150 3700 5150
+Wire Wire Line
+	3700 5150 3700 2650
+Wire Wire Line
+	3700 2650 3650 2650
 $EndSCHEMATC
