File: Hardware/kicad4ADSb0.1/ADSSBb0.1/ADSSBb0.1.kicad_pcb (KiCad board)
At the start: 2 copper layers, 18 parts, among them IC1 AD7856ANZ, J1 ICSP ARDUINO NANO, J2 Conn_01x04, J3 Conn_01x04, J4 Conn_01x04, J5 Conn_01x04, J6 Conn_01x04, J7 Conn_01x04, U1 MAX7375AXR405

Commit message: Kicad +
Kicad +
Parts:
- C5, IC1: moved to B.Cu
- J1: footprint Connector_PinHeader_2.54mm:PinHeader_2x03_P2.54mm_Vertical -> Connector_PinSocket_2.54mm:PinSocket_2x03_P2.54mm_Vertical; moved to B.Cu
- J2, J3, J4, J5, J6, J7: footprint Connector_PinHeader_2.54mm:PinHeader_1x04_P2.54mm_Vertical -> Connector_PinSocket_2.54mm:PinSocket_1x04_P2.54mm_Vertical
- moved C1 67.2 mm to (111.8, 95.2)
- moved J2 65.5 mm to (119.4, 114.3), turned to 90 degrees
- moved J3 61.9 mm to (119.4, 109.2), turned to 90 degrees
- moved C4 61.0 mm to (111.8, 105.4)
- moved J6 55.4 mm to (120.7, 87.6), turned to 90 degrees
- moved J7 54.3 mm to (120.9, 83.1), turned to 90 degrees
- moved C5 51.1 mm to (137.2, 114.3)
- moved U1 50.5 mm to (148.6, 87.6)
- moved J4 48.4 mm to (135.9, 87.6), turned to 90 degrees
- moved J5 47.9 mm to (135.9, 83.1), turned to 90 degrees
- moved R1 45.3 mm to (135.9, 106.7)
- moved C6 42.7 mm to (132.1, 111.8)
- moved C2 39.9 mm to (152.4, 92.7)
- moved C3 35.7 mm to (152.4, 99.1)
- moved C8 33.3 mm to (152.4, 105.4)
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