File: Hardware/kicad4ADSb0.1/ADSSBb0.1/ADSSBb0.1.sch (KiCad schematic (older format))
At the start: 12 parts, among them IC1 AD7856ANZ, J1 ICSP ARDUINO NANO, U1 MAX7375AXR405

Commit message: Kicad experiments
Kicad experiments
Parts:
- removed A1: Arduino_Nano_v3.x, Module:Arduino_Nano, symbol MCU_Module:Arduino_Nano_v3.x
- added C8: 0.1e-6, Capacitor_THT:CP_Radial_D4.0mm_P1.50mm, symbol Device:CP1_Small
- added J2, J3, J4, J5, J6, J7: Conn_01x04, Connector_PinHeader_2.54mm:PinHeader_1x04_P2.54mm_Vertical, symbol Connector_Generic:Conn_01x04
- C1, C2, C3, C4, C5, C6, C7: footprint (none) -> Capacitor_THT:CP_Radial_D4.0mm_P1.50mm
- IC1: footprint DIP794W56P254L3188H533Q24N -> Package_DIP:DIP-24_W10.16mm
- J1: footprint (none) -> Connector_PinHeader_2.54mm:PinHeader_2x03_P2.54mm_Vertical
- R1: footprint (none) -> Resistor_THT:R_Axial_DIN0204_L3.6mm_D1.6mm_P1.90mm_Vertical
Connections:
- net GND: now also J1.6 (Pin_6), C8.2, J2.2 (Pin_2), J3.2 (Pin_2), J4.2 (Pin_2), J5.2 (Pin_2), J6.2 (Pin_2), J7.2 (Pin_2)
- net at IC1.10 (AIN2): now also J3.3 (Pin_3)
- net at IC1.11 (AIN3): now also J4.3 (Pin_3)
- net at IC1.12 (AIN4): now also J5.3 (Pin_3)
- net at IC1.13 (AIN5): now also J6.3 (Pin_3)
- net at IC1.14 (AIN6): now also J7.3 (Pin_3)
- net 5V: now reaches C1.1, C2.1, IC1.5 (AVDD), R1.1, U1.1 (V+)
- net 5V: now also J1.2 (Pin_2), C8.1, J2.1 (Pin_1), J3.1 (Pin_1), J4.1 (Pin_1), J5.1 (Pin_1), J6.1 (Pin_1), J7.1 (Pin_1)
- net at IC1.9 (AIN1): now also J2.3 (Pin_3)

Commit message: Kicad +
Kicad +
Parts:
- J1: footprint Connector_PinHeader_2.54mm:PinHeader_2x03_P2.54mm_Vertical -> Connector_PinSocket_2.54mm:PinSocket_2x03_P2.54mm_Vertical
- J2, J3, J4, J5, J6, J7: footprint Connector_PinHeader_2.54mm:PinHeader_1x04_P2.54mm_Vertical -> Connector_PinSocket_2.54mm:PinSocket_1x04_P2.54mm_Vertical
Changed lines of the file:
@@
 F 0 "J1" V 4554 3880 50  0000 L CNN
 F 1 "ICSP ARDUINO NANO" V 4645 3880 50  0000 L CNN
-F 2 "Connector_PinHeader_2.54mm:PinHeader_2x03_P2.54mm_Vertical" H 4550 3700 50  0001 C CNN
+F 2 "Connector_PinSocket_2.54mm:PinSocket_2x03_P2.54mm_Vertical" H 4550 3700 50  0001 C CNN
 F 3 "~" H 4550 3700 50  0001 C CNN
 	1    4550 3700
@@
 F 0 "J2" H 1530 4292 50  0000 L CNN
 F 1 "Conn_01x04" H 1530 4201 50  0000 L CNN
-F 2 "Connector_PinHeader_2.54mm:PinHeader_1x04_P2.54mm_Vertical" H 1450 4300 50  0001 C CNN
+F 2 "Connector_PinSocket_2.54mm:PinSocket_1x04_P2.54mm_Vertical" H 1450 4300 50  0001 C CNN
 F 3 "~" H 1450 4300 50  0001 C CNN
 	1    1450 4300
@@
 F 0 "J3" H 1530 4942 50  0000 L CNN
 F 1 "Conn_01x04" H 1530 4851 50  0000 L CNN
-F 2 "Connector_PinHeader_2.54mm:PinHeader_1x04_P2.54mm_Vertical" H 1450 4950 50  0001 C CNN
+F 2 "Connector_PinSocket_2.54mm:PinSocket_1x04_P2.54mm_Vertical" H 1450 4950 50  0001 C CNN
 F 3 "~" H 1450 4950 50  0001 C CNN
 	1    1450 4950
@@
 F 0 "J4" H 1530 5642 50  0000 L CNN
 F 1 "Conn_01x04" H 1530 5551 50  0000 L CNN
-F 2 "Connector_PinHeader_2.54mm:PinHeader_1x04_P2.54mm_Vertical" H 1450 5650 50  0001 C CNN
+F 2 "Connector_PinSocket_2.54mm:PinSocket_1x04_P2.54mm_Vertical" H 1450 5650 50  0001 C CNN
 F 3 "~" H 1450 5650 50  0001 C CNN
 	1    1450 5650
@@
 F 0 "J5" H 2880 4292 50  0000 L CNN
 F 1 "Conn_01x04" H 2880 4201 50  0000 L CNN
-F 2 "Connector_PinHeader_2.54mm:PinHeader_1x04_P2.54mm_Vertical" H 2800 4300 50  0001 C CNN
+F 2 "Connector_PinSocket_2.54mm:PinSocket_1x04_P2.54mm_Vertical" H 2800 4300 50  0001 C CNN
 F 3 "~" H 2800 4300 50  0001 C CNN
 	1    2800 4300
@@
 F 0 "J6" H 2880 4942 50  0000 L CNN
 F 1 "Conn_01x04" H 2880 4851 50  0000 L CNN
-F 2 "Connector_PinHeader_2.54mm:PinHeader_1x04_P2.54mm_Vertical" H 2800 4950 50  0001 C CNN
+F 2 "Connector_PinSocket_2.54mm:PinSocket_1x04_P2.54mm_Vertical" H 2800 4950 50  0001 C CNN
 F 3 "~" H 2800 4950 50  0001 C CNN
 	1    2800 4950
@@
 F 0 "J7" H 2880 5642 50  0000 L CNN
 F 1 "Conn_01x04" H 2880 5551 50  0000 L CNN
-F 2 "Connector_PinHeader_2.54mm:PinHeader_1x04_P2.54mm_Vertical" H 2800 5650 50  0001 C CNN
+F 2 "Connector_PinSocket_2.54mm:PinSocket_1x04_P2.54mm_Vertical" H 2800 5650 50  0001 C CNN
 F 3 "~" H 2800 5650 50  0001 C CNN
 	1    2800 5650
